Commit message: Changes

File: description/robot.urdf.xacro (robot description, xacro)
@@ -1,31 +1,4 @@
 <?xml version="1.0"?>
 <robot xmlns:xacro="http://www.ros.org/wiki/xacro"  name="robot">
-<material name="white">
-    <color rgba="1 1 1 1" />
-</material>
-<material name="orange">
-    <color rgba="1 0.3 0.1 1" />
-</material>
-<material name="blue">
-    <color rgba="0.2 0.2 1 1" />
-</material>
-<material name="black">
-    <color rgba="0 0 0 1" />
-</material>
-<link name="base_link">
-</link>
-<joint name="chassis_joint" type="fixed">
-    <parent link="base link"/>
-    <child link="chassis"/>
-    <origin xyz="-0.1 0.0 0.0"/>
-</joint>
-<link name="chassis">
-    <visual>
-    <origin xyz="0.2 0 0.6"/>
-        <geometry>
-            <box size="0.4 0.4 0.12"/>
-        </geometry>
-        <material name="white"/>
-        </material>
-    </visual>
+    <xacro:include filename="robot core.xacro" />
 </robot>

Commit message: Change

File: description/robot.urdf.xacro (robot description, xacro)
@@ -1,4 +1,16 @@
 <?xml version="1.0"?>
 <robot xmlns:xacro="http://www.ros.org/wiki/xacro"  name="robot">
+    <material name="white">
+        <color rgba="1 1 1 1" />
+    </material>
+    <material name="orange">
+        <color rgba="1 0.3 0.1 1" />
+    </material>
+    <material name="blue">
+        <color rgba="0.2 0.2 1 1" />
+    </material>
+    <material name="black">
+        <color rgba="0 0 0 1" />
+    </material>
     <!-- <xacro:include filename="robot core.xacro" /> -->
 </robot>
